File: PCB/ShieldHallSensor/ShieldHallSensor.kicad_sch (KiCad schematic)
At the start: 8 parts, among them J1 Shield_Connector_Top_Left, J2 Shield_Connector_Bottom_Left, J3 Shield_Connector_Top_Right, J4 Shield_Connector_Bottom_Right, U1 HallLinearSensor

Commit message: Add power supply (wip) and update panel
Parts:
- J1, J2, J3, J4: LCSC (none) -> C2883469
Changed lines of the file:
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@@
+			)
+		)
+		(property "LCSC" "C2883469"
+			(at 91.44 87.63 0)
+			(effects
+				(font
+					(size 1.27 1.27)
+				)
+				(hide yes)
 			)
 		)
@@
 			)
 		)
+		(property "LCSC" "C2883469"
+			(at 142.24 87.63 0)
+			(effects
+				(font
+					(size 1.27 1.27)
+				)
+				(hide yes)
+			)
+		)
 		(pin "1"
 		)
@@
 			)
 		)
+		(property "LCSC" "C2883469"
+			(at 142.24 101.6 0)
+			(effects
+				(font
+					(size 1.27 1.27)
+				)
+				(hide yes)
+			)
+		)
 		(pin "1"
 		)
@@
 			(at 91.44 101.6 0)
 			(effects
+				(font
+					(size 1.27 1.27)
+				)
+				(hide yes)
+			)
+		)
+		(property "LCSC" "C2883469"
+			(at 91.44 101.6 0)
+			(effects
