File: PCB/Panel/SmartCubePanel.kicad_pcb (KiCad board)
At the start: 2 copper layers, 137.5 x 132 mm, 760 parts

Commit message: Add electrolytic bulk capacitors to modules and power supply
Parts:
- added M_1_C4: 470uF Electrolytic, CustomFootprints:CAP-SMD_BD6.3-L6.6-W6.6-FD, F.Cu at (105.6, 97.0)
- added M_2_C4: 470uF Electrolytic, CustomFootprints:CAP-SMD_BD6.3-L6.6-W6.6-FD, F.Cu at (105.6, 139.7)
- added M_3_C4: 470uF Electrolytic, CustomFootprints:CAP-SMD_BD6.3-L6.6-W6.6-FD, F.Cu at (148.3, 54.2)
- added M_4_C4: 470uF Electrolytic, CustomFootprints:CAP-SMD_BD6.3-L6.6-W6.6-FD, F.Cu at (148.3, 97.0)
- added M_5_C4: 470uF Electrolytic, CustomFootprints:CAP-SMD_BD6.3-L6.6-W6.6-FD, F.Cu at (148.3, 139.7)
- added PSU_0_C6: ElectrolyticCapacitorSMD, CustomFootprints:CAP-SMD_BD6.3-L6.6-W6.6-FD, F.Cu at (115.6, 41.9)
- added PSU_0_C7: ElectrolyticCapacitorSMD, CustomFootprints:CAP-SMD_BD6.3-L6.6-W6.6-FD, F.Cu at (120.6, 46.8)
- moved M_1_R5 1.14 mm to (112.9, 96.3)
- moved M_2_R5 1.14 mm to (112.9, 139.0)
- moved M_3_R5 1.14 mm to (155.6, 53.5)
- moved M_4_R5 1.14 mm to (155.6, 96.3)
- moved M_5_R5 1.14 mm to (155.6, 139.0)
Routing:
- net Board_0-GND: track 95.5 -> 98.9 mm, vias 17 -> 19
- net Board_2-GND: track 28.1 -> 29.9 mm, vias 11 -> 12
- net Board_1-GND: track 28.1 -> 29.9 mm, vias 11 -> 12
- net Board_5-GND: track 28.1 -> 29.9 mm, vias 11 -> 12
- net Board_3-GND: track 28.1 -> 29.9 mm, vias 11 -> 12
- net Board_4-GND: track 28.1 -> 29.9 mm, vias 11 -> 12
- net Board_1-/ShieldBottomLeft: track 19.8 -> 20.8 mm
- net Board_2-/ShieldBottomLeft: track 19.8 -> 20.8 mm
- net Board_5-/ShieldBottomLeft: track 19.8 -> 20.8 mm
- net Board_4-/ShieldBottomLeft: track 19.8 -> 20.8 mm
- net Board_3-/ShieldBottomLeft: track 19.8 -> 20.8 mm
- net Board_2-/DataBottom2: track 22.9 -> 23.9 mm
- net Board_5-/DataBottom2: track 22.9 -> 23.9 mm
- net Board_1-/DataBottom2: track 22.9 -> 23.9 mm
- net Board_3-/DataBottom2: track 22.9 -> 23.9 mm
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Other:
- board text added: "VCC"
- board text removed: "+5V"
